File: STM_Proto1.brd (EAGLE design)
At the start: 160 x 100 mm, 74 parts, among them Q1 8M, Q2 32748

Commit message: Update 1
Parts:
- removed U$4: STM32L152C6, STM32L152:LQFP48
- added IC1: LM358D, linear:SO08
- added R22: 30000, resistor:R0805
- added R23: 128405, resistor:R0805
- added R24: 119606, resistor:R0805
- added R25: 100000, resistor:R0805
- added STM32L152CBT6: STM32L152C6, STM32L152:LQFP48
- added SV1: (no value), con-lstb:MA03-1
- added TR1: (no value), discrete:R-7,5
- moved R18 71.5 mm to (-16.5, 99.1)
- moved C12 66.5 mm to (-16.5, 92.7)
- moved R11 66.5 mm to (-21.6, 92.7)
- moved D6 61.6 mm to (-81.3, 63.5)
- moved Q1 57.8 mm to (-25.4, 64.8)
- moved Q2 57.8 mm to (-16.5, 61.0)
- moved UART_DEBUG 57.4 mm to (-80.0, 72.4)
- moved D3 56.4 mm to (-21.6, 104.1)
- moved LED1 50.1 mm to (-16.5, 109.2)
- moved LED2 50.1 mm to (-22.9, 109.2)
- moved LED3 50.1 mm to (-29.2, 109.2)
- moved F1 45.5 mm to (-74.9, 45.7)
- moved F2 45.5 mm to (-85.1, 45.7)
- moved L2-FCM1608-0603 28.0 mm to (-87.6, 104.1)
- moved POWER 17.8 mm to (-54.6, 104.1)
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Connections:
- removed net RX_SIM: GSM1.3, UART_SIM.3
- removed net TX_SIM: GSM1.4, UART_SIM.2
- removed net USART_RX_STM: U$4.13
- removed net USART_TX_STM: U$4.12
- new net +3V3: R22.2, R23.2, SV1.3
- new net A0.0+: IC1.1, R25.1, SV1.1
- new net N$12: IC1.2, R23.1, R24.2, R25.2
- new net N$13: IC1.3, R22.1, TR1.2
- new net USART1_RX: STM32L152CBT6.31
- new net USART1_TX: STM32L152CBT6.30
- new net USART2_RX: GSM1.4, STM32L152CBT6.13, UART_SIM.2
- new net USART2_TX: GSM1.3, STM32L152CBT6.12, UART_SIM.3
- new net V+: IC1.8
- new net V-: IC1.4
- net 3.3V: now also STM32L152CBT6.24, STM32L152CBT6.36, STM32L152CBT6.48; no longer U$4.24, U$4.36, U$4.48
- net ADC_RES: now also STM32L152CBT6.18; no longer U$4.18
- net GND: now also R24.1, STM32L152CBT6.23, STM32L152CBT6.35, STM32L152CBT6.47, STM32L152CBT6.8, SV1.2, TR1.1; no longer U$4.23, U$4.35, U$4.47, U$4.8
- net N$2: now also STM32L152CBT6.5; no longer U$4.5
- net N$28: now also STM32L152CBT6.6; no longer U$4.6
- net N$29: now also STM32L152CBT6.4; no longer U$4.4
- net N$30: now also STM32L152CBT6.3; no longer U$4.3
- net N$31: now also STM32L152CBT6.9; no longer U$4.9
- net N$32: now also STM32L152CBT6.44; no longer U$4.44
- net N$35: now also STM32L152CBT6.20; no longer U$4.20
- net NRST: now also STM32L152CBT6.7; no longer U$4.7
- net SWCLK: now also STM32L152CBT6.37; no longer U$4.37
- net SWDAT: now also STM32L152CBT6.34; no longer U$4.34
