File: STM_Proto1.sch (EAGLE design)
At the start: 74 parts, among them Q1 8M, Q2 32748

Commit message: Update 1
Parts:
- removed U$4: STM32L152C6, STM32L152:STM32L152C6
- added IC1: LM358D, linear:LM358D
- added R22: 30000, resistor:R-EU_R0805
- added R23: 128405, resistor:R-EU_R0805
- added R24: 119606, resistor:R-EU_R0805
- added R25: 100000, resistor:R-EU_R0805
- added STM32L152CBT6: STM32L152C6, STM32L152:STM32L152C6
- added SV1: (no value), con-lstb:MA03-1
- added TR1: (no value), discrete:THERMISTOR_R-7,5
Connections:
- removed net RX_SIM: GSM1.RXD, UART_SIM.3
- removed net TX_SIM: GSM1.TXD, UART_SIM.2
- removed net USART_RX_STM: U$4.PA3
- removed net USART_TX_STM: U$4.PA2
- new net +3V3: R22.2, R23.2, SV1.3
- new net A0.0+: IC1A.OUT, R25.1, SV1.1
- new net N$12: IC1A.-IN, R23.1, R24.2, R25.2
- new net N$13: IC1A.+IN, R22.1, TR1.2
- new net USART1_RX: STM32L152CBT6.PA10
- new net USART1_TX: STM32L152CBT6.PA9
- new net USART2_RX: GSM1.TXD, STM32L152CBT6.PA3, UART_SIM.2
- new net USART2_TX: GSM1.RXD, STM32L152CBT6.PA2, UART_SIM.3
- net 3.3V: now also STM32L152CBT6.VDD_1, STM32L152CBT6.VDD_2, STM32L152CBT6.VDD_3; no longer U$4.VDD_1, U$4.VDD_2, U$4.VDD_3
- net ADC_RES: now also STM32L152CBT6.PB0; no longer U$4.PB0
- net GND: now also R24.1, STM32L152CBT6.VSSA, STM32L152CBT6.VSS_1, STM32L152CBT6.VSS_2, STM32L152CBT6.VSS_3, SV1.2, TR1.1; no longer U$4.VSSA, U$4.VSS_1, U$4.VSS_2, U$4.VSS_3
- net N$2: now also STM32L152CBT6.PH0; no longer U$4.PH0
- net N$28: now also STM32L152CBT6.PH1; no longer U$4.PH1
- net N$29: now also STM32L152CBT6.PC15_OSC_OUT; no longer U$4.PC15_OSC_OUT
- net N$30: now also STM32L152CBT6.PC14_OSC_IN; no longer U$4.PC14_OSC_IN
- net N$31: now also STM32L152CBT6.VDDA; no longer U$4.VDDA
- net N$32: now also STM32L152CBT6.BOOT0; no longer U$4.BOOT0
- net N$35: now also STM32L152CBT6.PB2; no longer U$4.PB2
- net NRST: now also STM32L152CBT6.NRST; no longer U$4.NRST
- net SWCLK: now also STM32L152CBT6.PA14; no longer U$4.PA14
- net SWDAT: now also STM32L152CBT6.PA13; no longer U$4.PA13
Other:
- moved on the sheet: AUDIO, C1, C10, C11, C12, C13, C14, C15, C16, C17, C18, C19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
